Commit message: updated simulation

File: src/ros_ur_driver/src/Universal_Robots_ROS2_Description/urdf/ur_macro.xacro (robot description, xacro)
@@ -341,5 +341,5 @@
          <safety_controller soft_lower_limit="${shoulder_pan_lower_limit + safety_pos_margin}" soft_upper_limit="${shoulder_pan_upper_limit - safety_pos_margin}" k_position="${safety_k_position}" k_velocity="0.0"/>
       </xacro:if>
-      <dynamics damping="0" friction="0"/>
+      <dynamics damping="0.7" friction="1.0"/>
     </joint>
     <joint name="${tf_prefix}shoulder_lift_joint" type="revolute">
@@ -353,5 +353,5 @@
          <safety_controller soft_lower_limit="${shoulder_lift_lower_limit + safety_pos_margin}" soft_upper_limit="${shoulder_lift_upper_limit - safety_pos_margin}" k_position="${safety_k_position}" k_velocity="0.0"/>
       </xacro:if>
-      <dynamics damping="0" friction="0"/>
+      <dynamics damping="0.7" friction="1.0"/>
     </joint>
     <joint name="${tf_prefix}elbow_joint" type="revolute">
@@ -365,5 +365,5 @@
          <safety_controller soft_lower_limit="${elbow_joint_lower_limit + safety_pos_margin}" soft_upper_limit="${elbow_joint_upper_limit - safety_pos_margin}" k_position="${safety_k_position}" k_velocity="0.0"/>
       </xacro:if>
-      <dynamics damping="0" friction="0"/>
+      <dynamics damping="0.7" friction="1.0"/>
     </joint>
     <joint name="${tf_prefix}wrist_1_joint" type="revolute">
@@ -377,5 +377,5 @@
          <safety_controller soft_lower_limit="${wrist_1_lower_limit + safety_pos_margin}" soft_upper_limit="${wrist_1_upper_limit - safety_pos_margin}" k_position="${safety_k_position}" k_velocity="0.0"/>
       </xacro:if>
-      <dynamics damping="0" friction="0"/>
+      <dynamics damping="0.7" friction="1.0"/>
     </joint>
     <joint name="${tf_prefix}wrist_2_joint" type="revolute">
@@ -389,5 +389,5 @@
          <safety_controller soft_lower_limit="${wrist_2_lower_limit + safety_pos_margin}" soft_upper_limit="${wrist_2_upper_limit - safety_pos_margin}" k_position="${safety_k_position}" k_velocity="0.0"/>
       </xacro:if>
-      <dynamics damping="0" friction="0"/>
+      <dynamics damping="0.7" friction="1.0"/>
     </joint>
     <joint name="${tf_prefix}wrist_3_joint" type="${wrist_3_joint_type}">
@@ -409,5 +409,5 @@
         </xacro:if>
       </xacro:unless>
-      <dynamics damping="0" friction="0"/>
+      <dynamics damping="0.7" friction="1.0"/>
     </joint>
     <link name="${tf_prefix}ft_frame"/>

File: src/ros_ur_driver/src/Universal_Robots_ROS2_Description/urdf/ur_mid360.urdf.xacro (robot description, xacro)
@@ -44,5 +44,5 @@
    <xacro:arg name="sim_gazebo" default="false" />
    <xacro:arg name="sim_ignition" default="false" />
-   <xacro:arg name="simulation_controllers" default="" />
+   <xacro:arg name="simulation_controllers" default="$(find ur_description)/config/ur_gazebo_controllers.yaml"/>
    <!-- initial position for simulations (Fake Hardware, Gazebo, Ignition) -->
    <xacro:arg name="initial_positions_file" default="$(find ur_description)/config/initial_positions.yaml"/>
@@ -71,8 +71,8 @@
        </collision>
      </link>
-     <joint name="ground_plane_joint" type="fixed">
-       <origin xyz="0 0 -0.01" rpy="0 0 0"/>
-       <parent link="world"/>
-       <child link="ground_plane"/>
+     <joint name="world_to_base" type="fixed">
+      <parent link="world"/>
+      <child link="ground_plane"/> <!-- replace with actual base link name -->
+      <origin xyz="0 0 0.05" rpy="0 0 0"/>
      </joint>
    </xacro:if>
@@ -117,8 +117,13 @@
      <origin xyz="0 0 0" rpy="0 0 0" />          <!-- position robot in the world -->
    </xacro:ur_robot>
-  <xacro:include filename="$(find ros2_livox_simulation)/urdf/mid360.xacro" />
-  <xacro:mid360 name="livox" parent="world" topic="mid360">
-    <origin xyz="0 2 0.025" rpy="0 0 0"/>
-  </xacro:mid360>
+    <joint name="world_to_lidar_mount" type="fixed">
+        <parent link="world"/>
+        <child link="lidar_mount"/>
+        <origin xyz="1.0 1.0 0.5" rpy="0 0 0"/>
+    </joint>
+    <xacro:include filename="$(find ros2_livox_simulation)/urdf/mid360.xacro"/>
+    <xacro:mid360 name="livox" parent="lidar_mount" topic="mid360">
+        <origin xyz="1.0 1.0 0.5" rpy="0 0 0"/>
+    </xacro:mid360>
    <xacro:if value="$(arg sim_gazebo)">
     <!-- Gazebo plugins -->
