Commit message: update with pcl

File: src/ros_ur_driver/src/Universal_Robots_ROS2_Description/urdf/ur_mid360.urdf.xacro (robot description, xacro)
@@ -117,12 +117,12 @@
      <origin xyz="0 0 0" rpy="0 0 0" />          <!-- position robot in the world -->
    </xacro:ur_robot>
-    <joint name="world_to_lidar_mount" type="fixed">
+    <!-- <joint name="world_to_lidar_mount" type="fixed">
         <parent link="world"/>
         <child link="lidar_mount"/>
         <origin xyz="1.0 1.0 0.5" rpy="0 0 0"/>
-    </joint>
+    </joint> -->
     <xacro:include filename="$(find ros2_livox_simulation)/urdf/mid360.xacro"/>
-    <xacro:mid360 name="livox" parent="lidar_mount" topic="mid360">
-        <origin xyz="1.0 1.0 0.5" rpy="0 0 0"/>
+    <xacro:mid360 name="livox" parent="world" topic="mid360">
+        <origin xyz="1.0 1.0 0.25" rpy="0 0 0"/>
     </xacro:mid360>
    <xacro:if value="$(arg sim_gazebo)">
